File: rhododendron.sch (KiCad schematic (older format))
At the start: 44 parts, among them J1 NEIGHBOR1, J2 NEIGHBOR2, J7 BONUS_ROW

Commit message: fix my inability to spell rhododendron :)
Parts:
- J?: symbol rhodadendron:USB-A-SHIELDED -> rhododendron:USB-A-SHIELDED; Manuf P/N (none) -> 87583-2010BLF
- U?: symbol rhodadendron:USB3343 -> rhododendron:USB3343
Changed lines of the file:
@@
 EESchema Schematic File Version 4
-LIBS:rhodadendron-cache
+LIBS:rhododendron-cache
 EELAYER 29 0
 EELAYER END
@@
 $EndComp
 $Comp
-L rhodadendron:USB3343 U?
+L rhododendron:USB3343 U?
 U 1 1 5CD28DED
 P 3200 2050
@@
 	6400 2550 6750 2550
 $Comp
-L rhodadendron:USB-A-SHIELDED J?
+L rhododendron:USB-A-SHIELDED J?
 U 1 1 5CE06275
 P 9200 3450
@@
 F 2 "" H 9200 3450 50  0001 C CNN
 F 3 "" H 9200 3450 50  0001 C CNN
+F 4 "87583-2010BLF" H 9200 3450 50  0001 C CNN "Manuf P/N"
 	1    9200 3450
 	1    0    0    -1
@@
 	0    -1   -1   0
 $EndComp
+Text Notes 13100 700  0    50   ~ 0
+mounting holes
 Wire Bus Line
 	2600 1500 2600 2750
-Text Notes 13100 700  0    50   ~ 0
-mounting holes
 $EndSCHEMATC
